Commit message: modify point cloud and camera srtting for double env

File: assets/robot/xarm6_description/xarm7_allegro_left.urdf (robot description, URDF)
Before this commit: robot xarm7, 31 links, 30 joints
Joints:
- joint gripper_base_joint: origin xyz=0.0 0 0.121 rpy=0 0 3.1416 -> xyz=0.03 0 0.045 rpy=3.1415926 -1.5707963267948966 0.0

File: assets/robot/xarm6_description/xarm7_allegro_right.urdf (robot description, URDF)
Before this commit: robot xarm7, 31 links, 30 joints
Links:
- link base_link: geometry collision box size=0.0408 0.1130 0.095; visual box size=0.015 0.085 0.03
Joints:
- joint gripper_base_joint: origin xyz=0.0 0 0.121 rpy=0 0 3.1416 -> xyz=-0.03 0 0.045 rpy=0 -1.5707963267948966 0.0

File: robot/xarm7_allegro_left.urdf (robot description, URDF)
Before this commit: robot xarm7, 31 links, 30 joints
Links:
- link base_link: geometry collision box size=0.0408 0.1130 0.095; visual box size=0.015 0.085 0.03
- link link_12.0: geometry collision box size=0.0358 0.034 0.0455; visual mesh filename=../allegro_hand_description/meshes/link_12.0_left.STL
Joints:
- joint gripper_base_joint: origin xyz=-0.03 0 0.045 rpy=0 -1.5707963267948966 0.0 -> xyz=0.0 0 0.121 rpy=0 0 3.1416
- joint joint_0.0: origin xyz=0 0.0435 -0.001542 rpy=-0.08726646255 0 0 -> xyz=0 -0.0435 -0.001542 rpy=0.08726646255 0 0
- joint joint_12.0: axis -1 0 0 -> +1 0 0; origin xyz=-0.0182 0.019333 -0.045987 rpy=0 -1.65806278845 -1.5707963259 -> xyz=-0.0182 -0.019333 -0.045987 rpy=0 -1.65806278845 1.5707963259
- joint joint_13.0: axis 0 0 1 -> 0 0 -1; origin xyz=-0.027 0.005 0.0399 -> xyz=-0.027 -0.005 0.0399
- joint joint_8.0: origin xyz=0 -0.0435 -0.001542 rpy=0.08726646255 0 0 -> xyz=0 0.0435 -0.001542 rpy=-0.08726646255 0 0

File: robot/xarm7_allegro_right.urdf (robot description, URDF)
Before this commit: robot xarm7, 31 links, 30 joints
Links:
- link base_link: geometry collision box size=0.0408 0.1130 0.095; visual mesh filename=../allegro_hand_description/meshes/base_link.STL
Joints:
- joint gripper_base_joint: origin xyz=-0.03 0 0.045 rpy=0 -1.5707963267948966 0.0 -> xyz=0.0 0 0.121 rpy=0 0 3.1416
